Commit message: more experimenting. need to figure out if it's cheating physics

File: models/pancake_flipper_massless_links.urdf (robot description, URDF)
Before this commit: robot pancake_flipper, 6 links, 6 joints
Links:
- link flipper: geometry collision box size=2 0.2 0.2; visual box size=2 0.2 0.2
